Commit message: Add gripper

File: assets/rox_diff_ur5e.urdf (robot description, URDF)
Before this commit: robot rox, 26 links, 25 joints
Links:
- added link gripper_mount_link
- added link robotiq_85_base_link, mass 6.6320197e-01; collision mesh filename=meshes/robotiq_description/collision/robotiq_base.stl; visual mesh filename=meshes/robotiq_description/visual/robotiq_base.dae
- added link robotiq_85_left_finger_link, mass 4.260376752e-02; collision mesh filename=meshes/robotiq_description/collision/left_finger.stl; visual mesh filename=meshes/robotiq_description/visual/left_finger.dae
- added link robotiq_85_left_finger_tip_link, mass 4.268588744e-02; collision mesh filename=meshes/robotiq_description/collision/left_finger_tip.stl; visual mesh filename=meshes/robotiq_description/visual/left_finger_tip.dae
- added link robotiq_85_left_inner_knuckle_link, mass 2.969376448e-02; collision mesh filename=meshes/robotiq_description/collision/left_inner_knuckle.stl; visual mesh filename=meshes/robotiq_description/visual/left_inner_knuckle.dae
- added link robotiq_85_left_knuckle_link, mass 1.384773208e-02; collision mesh filename=meshes/robotiq_description/collision/left_knuckle.stl; visual mesh filename=meshes/robotiq_description/visual/left_knuckle.dae
- added link robotiq_85_right_finger_link, mass 4.260376752000000e-02; collision mesh filename=meshes/robotiq_description/collision/right_finger.stl; visual mesh filename=meshes/robotiq_description/visual/right_finger.dae
- added link robotiq_85_right_finger_tip_link, mass 4.268588744e-02; collision mesh filename=meshes/robotiq_description/collision/right_finger_tip.stl; visual mesh filename=meshes/robotiq_description/visual/right_finger_tip.dae
- added link robotiq_85_right_inner_knuckle_link, mass 2.969376448e-02; collision mesh filename=meshes/robotiq_description/collision/right_inner_knuckle.stl; visual mesh filename=meshes/robotiq_description/visual/right_inner_knuckle.dae
- added link robotiq_85_right_knuckle_link, mass 1.384773208e-02; collision mesh filename=meshes/robotiq_description/collision/right_knuckle.stl; visual mesh filename=meshes/robotiq_description/visual/right_knuckle.dae
- added link ur_to_robotiq_link, mass 0.01; collision mesh filename=meshes/robotiq_description/collision/ur_to_robotiq_adapter.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; visual mesh filename=meshes/robotiq_description/visual/ur_to_robotiq_adapter.dae
Joints:
- added joint gripper_side_joint: type fixed, parent ur_to_robotiq_link, child gripper_mount_link, origin xyz=0 0 0.011 rpy=0 0 0
- added joint robotiq_85_base_joint: type fixed, parent gripper_mount_link, child robotiq_85_base_link, origin xyz=0 0 0 rpy=0 0 -1.5707963267948966
- added joint robotiq_85_left_finger_joint: type fixed, parent robotiq_85_left_knuckle_link, child robotiq_85_left_finger_link, origin xyz=0.03152616 0.0 -0.00376347 rpy=0 0 0
- added joint robotiq_85_left_finger_tip_joint: type continuous, parent robotiq_85_left_finger_link, child robotiq_85_left_finger_tip_link, origin xyz=0.00563134 0.0 0.04718515 rpy=0 0 0, axis 0 -1 0, mimic joint=robotiq_85_left_knuckle_joint multiplier=-1
- added joint robotiq_85_left_inner_knuckle_joint: type continuous, parent robotiq_85_base_link, child robotiq_85_left_inner_knuckle_link, origin xyz=0.0127 0.0 0.06142 rpy=0 0 0, axis 0 -1 0, mimic joint=robotiq_85_left_knuckle_joint
- added joint robotiq_85_left_knuckle_joint: type revolute, parent robotiq_85_base_link, child robotiq_85_left_knuckle_link, origin xyz=0.03060114 0.0 0.05490452 rpy=0 0 0, axis 0 -1 0, limit lower=0.0 upper=0.8 effort=50 velocity=0.5
- added joint robotiq_85_right_finger_joint: type fixed, parent robotiq_85_right_knuckle_link, child robotiq_85_right_finger_link, origin xyz=-0.03152616 0.0 -0.00376347 rpy=0 0 0
- added joint robotiq_85_right_finger_tip_joint: type continuous, parent robotiq_85_right_finger_link, child robotiq_85_right_finger_tip_link, origin xyz=-0.00563134 0.0 0.04718515 rpy=0 0 0, axis 0 -1 0, mimic joint=robotiq_85_left_knuckle_joint
- added joint robotiq_85_right_inner_knuckle_joint: type continuous, parent robotiq_85_base_link, child robotiq_85_right_inner_knuckle_link, origin xyz=-0.0127 0.0 0.06142 rpy=0 0 0, axis 0 -1 0, mimic joint=robotiq_85_left_knuckle_joint multiplier=-1
- added joint robotiq_85_right_knuckle_joint: type revolute, parent robotiq_85_base_link, child robotiq_85_right_knuckle_link, origin xyz=-0.03060114 0.0 0.05490452 rpy=0 0 0, axis 0 -1 0, limit lower=-0.8 upper=0.0 effort=50 velocity=0.5, mimic joint=robotiq_85_left_knuckle_joint multiplier=-1
- added joint ur_to_robotiq_joint: type fixed, parent ur5etool0, child ur_to_robotiq_link, origin xyz=0 0 0 rpy=0 0 1.5707963267948966

Commit message: feat: add grasp frame and plan to it instead of wrist_3
grasp_link aligns the gripper axes to the planning convention (Z out
of the gripper, X along finger travel) with a 0.134 m offset from
robotiq_85_base_link, so EE targets mean the grasp point, not the
wrist flange.

File: assets/rox_diff_ur5e.urdf (robot description, URDF)
Before this commit: robot rox, 37 links, 36 joints
Links:
- added link grasp_link
Joints:
- added joint grasp_link_joint: type fixed, parent robotiq_85_base_link, child grasp_link, origin xyz=0.0 0.0 0.134 rpy=0.0 0.0 3.141592653589793
